Commit message: Add per-joint enable flags and host-side impedance gains
- levion_system: per-joint enable params (left/right shoulder/elbow) so a
  single motor can be loaded without spurious CAN warnings
- ak80_8 macro: imp_kp/imp_kd params -> position interface runs the
  cubemars_hardware host-side impedance law
- point cubemars_hardware submodule at fork (impedance-host-side branch)

Co-Authored-By: Claude Opus 4.8 (1M context) <noreply@anthropic.com>

File: levion_arm_ros2_control/description/config/levion.property.xacro (robot description, xacro)
@@ -12,5 +12,9 @@
   <!-- Default -->
   <xacro:property name="default_joint_position_limit" value="${PI/2-SAFETY_OFFSET}"/>
+  <!-- Hardware driver vel_limit: value/10 * erpm_conversion → rad/s. Minimum 10 (= 1 rad/s). -->
   <xacro:property name="default_joint_velocity_limit" value="10"/>
+  <xacro:property name="default_joint_acceleration_limit" value="10"/>
+  <!-- URDF <limit velocity> used by JTC to reject fast trajectories (direct rad/s). -->
+  <xacro:property name="default_joint_urdf_velocity_limit" value="0.3"/>
   <xacro:property name="default_joint_effort_limit" value="10"/>
   <xacro:property name="shoulder_lower" value="-${default_joint_position_limit}"/>
@@ -24,4 +28,6 @@
   <xacro:property name="left_shoulder_upper" value="${shoulder_upper}"/>
   <xacro:property name="left_shoulder_velocity_limit" value="${default_joint_velocity_limit}"/>
+  <xacro:property name="left_shoulder_urdf_velocity_limit" value="${default_joint_urdf_velocity_limit}"/>
+  <xacro:property name="left_shoulder_acceleration_limit" value="${default_joint_acceleration_limit}"/>
   <xacro:property name="left_shoulder_effort_limit" value="${default_joint_effort_limit}"/>
   <xacro:property name="left_shoulder_enc_offset" value="${shoulder_enc_offset}"/>
@@ -29,4 +35,6 @@
   <xacro:property name="left_elbow_upper" value="${elbow_upper}"/>
   <xacro:property name="left_elbow_velocity_limit" value="${default_joint_velocity_limit}"/>
+  <xacro:property name="left_elbow_urdf_velocity_limit" value="${default_joint_urdf_velocity_limit}"/>
+  <xacro:property name="left_elbow_acceleration_limit" value="${default_joint_acceleration_limit}"/>
   <xacro:property name="left_elbow_effort_limit" value="${default_joint_effort_limit}"/>
   <xacro:property name="left_elbow_enc_offset" value="${elbow_enc_offset}"/>
@@ -35,4 +43,6 @@
   <xacro:property name="right_shoulder_upper" value="${-shoulder_lower}"/>
   <xacro:property name="right_shoulder_velocity_limit" value="${default_joint_velocity_limit}"/>
+  <xacro:property name="right_shoulder_urdf_velocity_limit" value="${default_joint_urdf_velocity_limit}"/>
+  <xacro:property name="right_shoulder_acceleration_limit" value="${default_joint_acceleration_limit}"/>
   <xacro:property name="right_shoulder_effort_limit" value="${default_joint_effort_limit}"/>
   <xacro:property name="right_shoulder_enc_offset" value="${-shoulder_enc_offset}"/>
@@ -40,4 +50,6 @@
   <xacro:property name="right_elbow_upper" value="${-elbow_lower}"/>
   <xacro:property name="right_elbow_velocity_limit" value="${default_joint_velocity_limit}"/>
+  <xacro:property name="right_elbow_urdf_velocity_limit" value="${default_joint_urdf_velocity_limit}"/>
+  <xacro:property name="right_elbow_acceleration_limit" value="${default_joint_acceleration_limit}"/>
   <xacro:property name="right_elbow_effort_limit" value="${default_joint_effort_limit}"/>
   <xacro:property name="right_elbow_enc_offset" value="${-elbow_enc_offset}"/>

File: levion_arm_ros2_control/description/ros2_control/ak80_8.macros.xacro (robot description, xacro)
@@ -1,5 +1,5 @@
 <?xml version="1.0"?>
 <robot xmlns:xacro="http://ros.org/wiki/xacro">
-  <xacro:macro name="ak80_8_ros2_control" params="joint_name can_id pos_min:=0.349 pos_max:=2.615 vel_limit:=10 effort_limit:=10 enc_off:=0">
+  <xacro:macro name="ak80_8_ros2_control" params="joint_name can_id pos_min:=0.349 pos_max:=2.615 vel_limit:=10 acc_limit:=10 effort_limit:=10 enc_off:=0 imp_kp:='' imp_kd:=0">
     <joint name="${joint_name}">
       <!-- ros2 control basic setting -->
@@ -25,8 +25,16 @@
       <param name="gear_ratio">8</param>
       <param name="kt">0.199</param>
+      <param name="vel_limit">${vel_limit}</param>
+      <param name="acc_limit">${acc_limit}</param>
       <!-- levion arm settings -->
       <param name="pos_limit_min">${pos_min}</param>
       <param name="pos_limit_max">${pos_max}</param>
       <param name="enc_off">${enc_off}</param>
+      <!-- host-side impedance: set imp_kp (and optionally imp_kd) to realize the
+           position command interface as an impedance law over the current loop -->
+      <xacro:if value="${imp_kp != ''}">
+        <param name="imp_kp">${imp_kp}</param>
+        <param name="imp_kd">${imp_kd}</param>
+      </xacro:if>
     </joint>
   </xacro:macro>

File: levion_arm_ros2_control/description/ros2_control/levion_arm.ros2_control.xacro (robot description, xacro)
@@ -1,7 +1,8 @@
 <?xml version="1.0"?>
 <robot xmlns:xacro="http://www.ros.org/wiki/xacro">
-<xacro:macro name="levion_system" params="name prefix left_arm:=true right_arm:=false hw_plugin:='real'"> <!-- real/mujoco-->
+<xacro:macro name="levion_system" params="name prefix left_arm:=true right_arm:=false left_shoulder:=true left_elbow:=true right_shoulder:=true right_elbow:=true hw_plugin:='real'"> <!-- real/rsl_servo/mujoco/gazebo -->
 <!-- include macros -->
 <xacro:include filename="$(find levion_arm_ros2_control)/ros2_control/ak80_8.macros.xacro"/>
+<xacro:include filename="$(find cubemars_servo_hardware)/ros2_control/ak80_8_servo.macros.xacro"/>
 <xacro:include filename="$(find levion_arm_ros2_control)/config/levion.property.xacro"/>
 <ros2_control name="${name}" type="system">
@@ -9,4 +10,10 @@
     <hardware>
       <plugin>cubemars_hardware/CubeMarsSystemHardware</plugin>
+      <param name="can_interface">can0</param>
+    </hardware>
+  </xacro:if>
+  <xacro:if value="${hw_plugin == 'rsl_servo'}">
+    <hardware>
+      <plugin>cubemars_servo_hardware/ServoHardwareInterface</plugin>
       <param name="can_interface">can0</param>
     </hardware>
@@ -23,13 +30,19 @@
   </xacro:if>
   <!-- Left arm -->
-  <xacro:if value="${left_arm}">
+  <xacro:if value="${left_arm and hw_plugin != 'rsl_servo'}">
+    <xacro:if value="${left_shoulder}">
     <xacro:ak80_8_ros2_control
       joint_name="${prefix}left_shoulder_joint"
-      can_id="104"
+      can_id="204"
       pos_min="${left_shoulder_lower}"
       pos_max="${left_shoulder_upper}"
       vel_limit="${left_shoulder_velocity_limit}"
+      acc_limit="${left_shoulder_acceleration_limit}"
       effort_limit="${left_shoulder_effort_limit}"
-      enc_off="${left_shoulder_enc_offset}"/>
+      enc_off="${left_shoulder_enc_offset}"
+      imp_kp="2.0"
+      imp_kd="0.9"/>
+    </xacro:if>
+    <xacro:if value="${left_elbow}">
     <xacro:ak80_8_ros2_control
       joint_name="${prefix}left_elbow_joint"
@@ -38,17 +51,52 @@
       pos_max="${left_elbow_upper}"
       vel_limit="${left_elbow_velocity_limit}"
+      acc_limit="${left_elbow_acceleration_limit}"
+      effort_limit="${left_elbow_effort_limit}"
+      enc_off="${left_elbow_enc_offset}"
+      imp_kp="2.0"
+      imp_kd="0.9"/>
+    </xacro:if>
+  </xacro:if>
+  <!-- Left arm (RSL servo drivers; vel/acc properties are value/10 = rad/s) -->
+  <xacro:if value="${left_arm and hw_plugin == 'rsl_servo'}">
+    <xacro:if value="${left_shoulder}">
+    <xacro:ak80_8_servo_ros2_control
+      joint_name="${prefix}left_shoulder_joint"
+      can_id="204"
+      pos_min="${left_shoulder_lower}"
+      pos_max="${left_shoulder_upper}"
+      vel_limit="${left_shoulder_velocity_limit/10}"
+      acc_limit="${left_shoulder_acceleration_limit/10}"
+      effort_limit="${left_shoulder_effort_limit}"
+      enc_off="${left_shoulder_enc_offset}"/>
+    </xacro:if>
+    <xacro:if value="${left_elbow}">
+    <xacro:ak80_8_servo_ros2_control
+      joint_name="${prefix}left_elbow_joint"
+      can_id="105"
+      pos_min="${left_elbow_lower}"
+      pos_max="${left_elbow_upper}"
+      vel_limit="${left_elbow_velocity_limit/10}"
+      acc_limit="${left_elbow_acceleration_limit/10}"
       effort_limit="${left_elbow_effort_limit}"
       enc_off="${left_elbow_enc_offset}"/>
+    </xacro:if>
   </xacro:if>
   <!-- Right arm -->
-  <xacro:if value="${right_arm}">
+  <xacro:if value="${right_arm and hw_plugin != 'rsl_servo'}">
+    <xacro:if value="${right_shoulder}">
     <xacro:ak80_8_ros2_control
       joint_name="${prefix}right_shoulder_joint"
-      can_id="204"
+      can_id="104"
       pos_min="${right_shoulder_lower}"
       pos_max="${right_shoulder_upper}"
       vel_limit="${right_shoulder_velocity_limit}"
+      acc_limit="${right_shoulder_acceleration_limit}"
       effort_limit="${right_shoulder_effort_limit}"
-      enc_off="${right_shoulder_enc_offset}"/>
+      enc_off="${right_shoulder_enc_offset}"
+      imp_kp="1.0"
+      imp_kd="0.1"/>
+    </xacro:if>
+    <xacro:if value="${right_elbow}">
     <xacro:ak80_8_ros2_control
       joint_name="${prefix}right_elbow_joint"
@@ -57,6 +105,35 @@
       pos_max="${right_elbow_upper}"
       vel_limit="${right_elbow_velocity_limit}"
+      acc_limit="${right_elbow_acceleration_limit}"
+      effort_limit="${right_elbow_effort_limit}"
+      enc_off="${right_elbow_enc_offset}"
+      imp_kp="2.0"
+      imp_kd="0.9"/>
+    </xacro:if>
+  </xacro:if>
+  <!-- Right arm (RSL servo drivers; vel/acc properties are value/10 = rad/s) -->
+  <xacro:if value="${right_arm and hw_plugin == 'rsl_servo'}">
+    <xacro:if value="${right_shoulder}">
+    <xacro:ak80_8_servo_ros2_control
+      joint_name="${prefix}right_shoulder_joint"
+      can_id="104"
+      pos_min="${right_shoulder_lower}"
+      pos_max="${right_shoulder_upper}"
+      vel_limit="${right_shoulder_velocity_limit/10}"
+      acc_limit="${right_shoulder_acceleration_limit/10}"
+      effort_limit="${right_shoulder_effort_limit}"
+      enc_off="${right_shoulder_enc_offset}"/>
+    </xacro:if>
+    <xacro:if value="${right_elbow}">
+    <xacro:ak80_8_servo_ros2_control
+      joint_name="${prefix}right_elbow_joint"
+      can_id="205"
+      pos_min="${right_elbow_lower}"
+      pos_max="${right_elbow_upper}"
+      vel_limit="${right_elbow_velocity_limit/10}"
+      acc_limit="${right_elbow_acceleration_limit/10}"
       effort_limit="${right_elbow_effort_limit}"
       enc_off="${right_elbow_enc_offset}"/>
+    </xacro:if>
   </xacro:if>
 </ros2_control>

File: levion_arm_ros2_control/description/urdf/levion_arm.macros.xacro (robot description, xacro)
@@ -7,9 +7,9 @@
     <xacro:property name="lr_shoulder_lower" default="${left_shoulder_lower}" />
     <xacro:property name="lr_shoulder_upper" default="${left_shoulder_upper}" />
-    <xacro:property name="lr_shoulder_vel" default="${left_shoulder_velocity_limit}" />
+    <xacro:property name="lr_shoulder_vel" default="${left_shoulder_urdf_velocity_limit}" />
     <xacro:property name="lr_shoulder_effort" default="${left_shoulder_effort_limit}" />
     <xacro:property name="lr_elbow_lower" default="${left_elbow_lower}" />
     <xacro:property name="lr_elbow_upper" default="${left_elbow_upper}" />
-    <xacro:property name="lr_elbow_vel" default="${left_elbow_velocity_limit}" />
+    <xacro:property name="lr_elbow_vel" default="${left_elbow_urdf_velocity_limit}" />
     <xacro:property name="lr_elbow_effort" default="${left_elbow_effort_limit}" />
   </xacro:if>
@@ -17,9 +17,9 @@
     <xacro:property name="lr_shoulder_lower" default="${right_shoulder_lower}" />
     <xacro:property name="lr_shoulder_upper" default="${right_shoulder_upper}" />
-    <xacro:property name="lr_shoulder_vel" default="${right_shoulder_velocity_limit}" />
+    <xacro:property name="lr_shoulder_vel" default="${right_shoulder_urdf_velocity_limit}" />
     <xacro:property name="lr_shoulder_effort" default="${right_shoulder_effort_limit}" />
     <xacro:property name="lr_elbow_lower" default="${right_elbow_lower}" />
     <xacro:property name="lr_elbow_upper" default="${right_elbow_upper}" />
-    <xacro:property name="lr_elbow_vel" default="${right_elbow_velocity_limit}" />
+    <xacro:property name="lr_elbow_vel" default="${right_elbow_urdf_velocity_limit}" />
     <xacro:property name="lr_elbow_effort" default="${right_elbow_effort_limit}" />
   </xacro:if>
