Commit message: Update leptrino submodule pointer and arm hardware properties

File: levion_arm_ros2_control/description/config/levion.property.xacro (robot description, xacro)
@@ -21,6 +21,10 @@
   <xacro:property name="shoulder_upper" value="${default_joint_position_limit}"/>
   <xacro:property name="shoulder_enc_offset" value="0"/>
-  <xacro:property name="elbow_lower" value="${-2.615+SAFETY_OFFSET}"/>
-  <xacro:property name="elbow_upper" value="${-0.349-SAFETY_OFFSET}"/>
+  <!-- Elbow position limits (rad). Left and right arms are physically different,
+       so each side has its own measured range. -->
+  <xacro:property name="left_elbow_lower_limit"  value="${-3.4+SAFETY_OFFSET}"/>
+  <xacro:property name="left_elbow_upper_limit"  value="${-1.2-SAFETY_OFFSET}"/>
+  <xacro:property name="right_elbow_lower_limit" value="${1.5+SAFETY_OFFSET}"/>
+  <xacro:property name="right_elbow_upper_limit" value="${3.7-SAFETY_OFFSET}"/>
   <xacro:property name="elbow_enc_offset" value="0.349"/>
   <!-- Left joints -->
@@ -32,6 +36,6 @@
   <xacro:property name="left_shoulder_effort_limit" value="${default_joint_effort_limit}"/>
   <xacro:property name="left_shoulder_enc_offset" value="${shoulder_enc_offset}"/>
-  <xacro:property name="left_elbow_lower" value="${elbow_lower}"/>
-  <xacro:property name="left_elbow_upper" value="${elbow_upper}"/>
+  <xacro:property name="left_elbow_lower" value="${left_elbow_lower_limit}"/>
+  <xacro:property name="left_elbow_upper" value="${left_elbow_upper_limit}"/>
   <xacro:property name="left_elbow_velocity_limit" value="${default_joint_velocity_limit}"/>
   <xacro:property name="left_elbow_urdf_velocity_limit" value="${default_joint_urdf_velocity_limit}"/>
@@ -47,6 +51,7 @@
   <xacro:property name="right_shoulder_effort_limit" value="${default_joint_effort_limit}"/>
   <xacro:property name="right_shoulder_enc_offset" value="${-shoulder_enc_offset}"/>
-  <xacro:property name="right_elbow_lower" value="${-elbow_upper}"/>
-  <xacro:property name="right_elbow_upper" value="${-elbow_lower}"/>
+  <!-- Right elbow uses its own measured range (not mirrored from the left) -->
+  <xacro:property name="right_elbow_lower" value="${right_elbow_lower_limit}"/>
+  <xacro:property name="right_elbow_upper" value="${right_elbow_upper_limit}"/>
   <xacro:property name="right_elbow_velocity_limit" value="${default_joint_velocity_limit}"/>
   <xacro:property name="right_elbow_urdf_velocity_limit" value="${default_joint_urdf_velocity_limit}"/>

File: levion_arm_ros2_control/description/ros2_control/ak80_8.macros.xacro (robot description, xacro)
@@ -1,5 +1,5 @@
 <?xml version="1.0"?>
 <robot xmlns:xacro="http://ros.org/wiki/xacro">
-  <xacro:macro name="ak80_8_ros2_control" params="joint_name can_id pos_min:=0.349 pos_max:=2.615 vel_limit:=10 acc_limit:=10 effort_limit:=10 enc_off:=0 imp_kp:='' imp_kd:=0">
+  <xacro:macro name="ak80_8_ros2_control" params="joint_name can_id pos_min:=0.349 pos_max:=2.615 vel_limit:=10 acc_limit:=10 effort_limit:=10 enc_off:=0 imp_kp:='' imp_kd:=0 use_speed_loop:=true">
     <joint name="${joint_name}">
       <!-- ros2 control basic setting -->
@@ -25,6 +25,13 @@
       <param name="gear_ratio">8</param>
       <param name="kt">0.199</param>
-      <param name="vel_limit">${vel_limit}</param>
-      <param name="acc_limit">${acc_limit}</param>
+      <!-- Setting BOTH vel_limit and acc_limit selects Position-Speed Loop (servo mode 6),
+           where the motor runs its own trapezoidal planner to each target. That fights a
+           joint_trajectory_controller streaming setpoints (oscillation). Set
+           use_speed_loop=false to omit them and use plain Position Loop (mode 4), which
+           tracks streamed setpoints smoothly. (Ignored when imp_kp is set -> impedance.) -->
+      <xacro:if value="${use_speed_loop}">
+        <param name="vel_limit">${vel_limit}</param>
+        <param name="acc_limit">${acc_limit}</param>
+      </xacro:if>
       <!-- levion arm settings -->
       <param name="pos_limit_min">${pos_min}</param>

File: levion_arm_ros2_control/description/ros2_control/levion_arm.ros2_control.xacro (robot description, xacro)
@@ -1,8 +1,7 @@
 <?xml version="1.0"?>
 <robot xmlns:xacro="http://www.ros.org/wiki/xacro">
-<xacro:macro name="levion_system" params="name prefix left_arm:=true right_arm:=false left_shoulder:=true left_elbow:=true right_shoulder:=true right_elbow:=true hw_plugin:='real'"> <!-- real/rsl_servo/mujoco/gazebo -->
+<xacro:macro name="levion_system" params="name prefix left_arm:=true right_arm:=false left_shoulder:=true left_elbow:=true right_shoulder:=true right_elbow:=true hw_plugin:='real'"> <!-- real/mujoco/gazebo -->
 <!-- include macros -->
 <xacro:include filename="$(find levion_arm_ros2_control)/ros2_control/ak80_8.macros.xacro"/>
-<xacro:include filename="$(find cubemars_servo_hardware)/ros2_control/ak80_8_servo.macros.xacro"/>
 <xacro:include filename="$(find levion_arm_ros2_control)/config/levion.property.xacro"/>
 <ros2_control name="${name}" type="system">
@@ -10,10 +9,4 @@
     <hardware>
       <plugin>cubemars_hardware/CubeMarsSystemHardware</plugin>
-      <param name="can_interface">can0</param>
-    </hardware>
-  </xacro:if>
-  <xacro:if value="${hw_plugin == 'rsl_servo'}">
-    <hardware>
-      <plugin>cubemars_servo_hardware/ServoHardwareInterface</plugin>
       <param name="can_interface">can0</param>
     </hardware>
@@ -30,9 +23,9 @@
   </xacro:if>
   <!-- Left arm -->
-  <xacro:if value="${left_arm and hw_plugin != 'rsl_servo'}">
+  <xacro:if value="${left_arm}">
     <xacro:if value="${left_shoulder}">
     <xacro:ak80_8_ros2_control
       joint_name="${prefix}left_shoulder_joint"
-      can_id="204"
+      can_id="93"
       pos_min="${left_shoulder_lower}"
       pos_max="${left_shoulder_upper}"
@@ -41,6 +34,6 @@
       effort_limit="${left_shoulder_effort_limit}"
       enc_off="${left_shoulder_enc_offset}"
-      imp_kp="2.0"
-      imp_kd="0.9"/>
+      imp_kp="1.0"
+      imp_kd="0.1"/>
     </xacro:if>
     <xacro:if value="${left_elbow}">
@@ -54,35 +47,10 @@
       effort_limit="${left_elbow_effort_limit}"
       enc_off="${left_elbow_enc_offset}"
-      imp_kp="2.0"
-      imp_kd="0.9"/>
-    </xacro:if>
-  </xacro:if>
-  <!-- Left arm (RSL servo drivers; vel/acc properties are value/10 = rad/s) -->
-  <xacro:if value="${left_arm and hw_plugin == 'rsl_servo'}">
-    <xacro:if value="${left_shoulder}">
-    <xacro:ak80_8_servo_ros2_control
-      joint_name="${prefix}left_shoulder_joint"
-      can_id="204"
-      pos_min="${left_shoulder_lower}"
-      pos_max="${left_shoulder_upper}"
-      vel_limit="${left_shoulder_velocity_limit/10}"
-      acc_limit="${left_shoulder_acceleration_limit/10}"
-      effort_limit="${left_shoulder_effort_limit}"
-      enc_off="${left_shoulder_enc_offset}"/>
-    </xacro:if>
-    <xacro:if value="${left_elbow}">
-    <xacro:ak80_8_servo_ros2_control
-      joint_name="${prefix}left_elbow_joint"
-      can_id="105"
-      pos_min="${left_elbow_lower}"
-      pos_max="${left_elbow_upper}"
-      vel_limit="${left_elbow_velocity_limit/10}"
-      acc_limit="${left_elbow_acceleration_limit/10}"
-      effort_limit="${left_elbow_effort_limit}"
-      enc_off="${left_elbow_enc_offset}"/>
+      imp_kp="0.5"
+      imp_kd="0.05"/>
     </xacro:if>
   </xacro:if>
   <!-- Right arm -->
-  <xacro:if value="${right_arm and hw_plugin != 'rsl_servo'}">
+  <xacro:if value="${right_arm}">
     <xacro:if value="${right_shoulder}">
     <xacro:ak80_8_ros2_control
@@ -108,31 +76,7 @@
       effort_limit="${right_elbow_effort_limit}"
       enc_off="${right_elbow_enc_offset}"
-      imp_kp="2.0"
-      imp_kd="0.9"/>
-    </xacro:if>
-  </xacro:if>
-  <!-- Right arm (RSL servo drivers; vel/acc properties are value/10 = rad/s) -->
-  <xacro:if value="${right_arm and hw_plugin == 'rsl_servo'}">
-    <xacro:if value="${right_shoulder}">
-    <xacro:ak80_8_servo_ros2_control
-      joint_name="${prefix}right_shoulder_joint"
-      can_id="104"
-      pos_min="${right_shoulder_lower}"
-      pos_max="${right_shoulder_upper}"
-      vel_limit="${right_shoulder_velocity_limit/10}"
-      acc_limit="${right_shoulder_acceleration_limit/10}"
-      effort_limit="${right_shoulder_effort_limit}"
-      enc_off="${right_shoulder_enc_offset}"/>
-    </xacro:if>
-    <xacro:if value="${right_elbow}">
-    <xacro:ak80_8_servo_ros2_control
-      joint_name="${prefix}right_elbow_joint"
-      can_id="205"
-      pos_min="${right_elbow_lower}"
-      pos_max="${right_elbow_upper}"
-      vel_limit="${right_elbow_velocity_limit/10}"
-      acc_limit="${right_elbow_acceleration_limit/10}"
-      effort_limit="${right_elbow_effort_limit}"
-      enc_off="${right_elbow_enc_offset}"/>
+      use_speed_loop="false"
+      imp_kp="0.5"
+      imp_kd="0.05"/>
     </xacro:if>
   </xacro:if>
